Commit message: Added convex mesh tags for URDF version 2 support

File: abb_irb6700_support/urdf/irb6700_200_260_macro.xacro (robot description, xacro)
@@ -15,5 +15,5 @@
         <origin xyz="0 0 0" rpy="0 0 0" />
         <geometry>
-          <mesh filename="package://abb_irb6700_support/meshes/irb6700/collision/base_link.stl" />
+          <convex_mesh filename="package://abb_irb6700_support/meshes/irb6700/collision/base_link.stl" convert="true"/>
         </geometry>
         <xacro:material_abb_yellow/>
@@ -31,5 +31,5 @@
         <origin xyz="0 0 0" rpy="0 0 0" />
         <geometry>
-          <mesh filename="package://abb_irb6700_support/meshes/irb6700/collision/link_1.stl" />
+          <convex_mesh filename="package://abb_irb6700_support/meshes/irb6700/collision/link_1.stl" convert="true"/>
         </geometry>
         <xacro:material_abb_yellow/>
@@ -47,5 +47,5 @@
         <origin xyz="0 0 0" rpy="0 0 0" />
         <geometry>
-          <mesh filename="package://abb_irb6700_support/meshes/irb6700/collision/cylinder.stl" />
+          <convex_mesh filename="package://abb_irb6700_support/meshes/irb6700/collision/cylinder.stl" convert="true"/>
         </geometry>
         <xacro:material_abb_yellow/>
@@ -63,5 +63,5 @@
         <origin xyz="0 0 0" rpy="0 0 0" />
         <geometry>
-          <mesh filename="package://abb_irb6700_support/meshes/irb6700/collision/piston.stl" />
+          <convex_mesh filename="package://abb_irb6700_support/meshes/irb6700/collision/piston.stl" convert="true"/>
         </geometry>
         <xacro:material_abb_yellow/>
@@ -79,5 +79,5 @@
         <origin xyz="0 0 0" rpy="0 0 0" />
         <geometry>
-          <mesh filename="package://abb_irb6700_support/meshes/irb6700_200_260/collision/link_2.stl" />
+          <convex_mesh filename="package://abb_irb6700_support/meshes/irb6700_200_260/collision/link_2.stl" convert="true"/>
         </geometry>
         <xacro:material_abb_yellow/>
@@ -95,5 +95,5 @@
         <origin xyz="0 0 0" rpy="0 0 0" />
         <geometry>
-          <mesh filename="package://abb_irb6700_support/meshes/irb6700_200_260/collision/link_3.stl" />
+          <convex_mesh filename="package://abb_irb6700_support/meshes/irb6700_200_260/collision/link_3.stl" convert="true"/>
         </geometry>
         <xacro:material_abb_yellow/>
@@ -111,5 +111,5 @@
         <origin xyz="0 0 0" rpy="0 0 0" />
         <geometry>
-          <mesh filename="package://abb_irb6700_support/meshes/irb6700_200_260/collision/link_4.stl" />
+          <convex_mesh filename="package://abb_irb6700_support/meshes/irb6700_200_260/collision/link_4.stl" convert="true"/>
         </geometry>
         <xacro:material_abb_yellow/>
@@ -127,5 +127,5 @@
         <origin xyz="0 0 0" rpy="0 0 0" />
         <geometry>
-          <mesh filename="package://abb_irb6700_support/meshes/irb6700/collision/link_5.stl" />
+          <convex_mesh filename="package://abb_irb6700_support/meshes/irb6700/collision/link_5.stl" convert="true"/>
         </geometry>
         <xacro:material_abb_yellow/>
@@ -143,5 +143,5 @@
         <origin xyz="0 0 0" rpy="0 0 0" />
         <geometry>
-          <mesh filename="package://abb_irb6700_support/meshes/irb6700/collision/link_6.stl" />
+          <convex_mesh filename="package://abb_irb6700_support/meshes/irb6700/collision/link_6.stl" convert="true"/>
         </geometry>
         <xacro:material_abb_yellow/>

File: abb_irb6700_support/urdf/irb6700_235_265_macro.xacro (robot description, xacro)
@@ -15,5 +15,5 @@
         <origin xyz="0 0 0" rpy="0 0 0" />
         <geometry>
-          <mesh filename="package://abb_irb6700_support/meshes/irb6700/collision/base_link.stl" />
+          <convex_mesh filename="package://abb_irb6700_support/meshes/irb6700/collision/base_link.stl" convert="true"/>
         </geometry>
         <xacro:material_abb_yellow/>
@@ -31,5 +31,5 @@
         <origin xyz="0 0 0" rpy="0 0 0" />
         <geometry>
-          <mesh filename="package://abb_irb6700_support/meshes/irb6700/collision/link_1.stl" />
+          <convex_mesh filename="package://abb_irb6700_support/meshes/irb6700/collision/link_1.stl" convert="true"/>
         </geometry>
         <xacro:material_abb_yellow/>
@@ -47,5 +47,5 @@
         <origin xyz="0 0 0" rpy="0 0 0" />
         <geometry>
-          <mesh filename="package://abb_irb6700_support/meshes/irb6700/collision/cylinder.stl" />
+          <convex_mesh filename="package://abb_irb6700_support/meshes/irb6700/collision/cylinder.stl" convert="true"/>
         </geometry>
         <xacro:material_abb_yellow/>
@@ -63,5 +63,5 @@
         <origin xyz="0 0 0" rpy="0 0 0" />
         <geometry>
-          <mesh filename="package://abb_irb6700_support/meshes/irb6700/collision/piston.stl" />
+          <convex_mesh filename="package://abb_irb6700_support/meshes/irb6700/collision/piston.stl" convert="true"/>
         </geometry>
         <xacro:material_abb_yellow/>
@@ -79,5 +79,5 @@
         <origin xyz="0 0 0" rpy="0 0 0" />
         <geometry>
-          <mesh filename="package://abb_irb6700_support/meshes/irb6700_235_265/collision/link_2.stl" />
+          <convex_mesh filename="package://abb_irb6700_support/meshes/irb6700_235_265/collision/link_2.stl" convert="true"/>
         </geometry>
         <xacro:material_abb_yellow/>
@@ -95,5 +95,5 @@
         <origin xyz="0 0 0" rpy="0 0 0" />
         <geometry>
-          <mesh filename="package://abb_irb6700_support/meshes/irb6700_235_265/collision/link_3.stl" />
+          <convex_mesh filename="package://abb_irb6700_support/meshes/irb6700_235_265/collision/link_3.stl" convert="true"/>
         </geometry>
         <xacro:material_abb_yellow/>
@@ -111,5 +111,5 @@
         <origin xyz="0 0 0" rpy="0 0 0" />
         <geometry>
-          <mesh filename="package://abb_irb6700_support/meshes/irb6700_235_265/collision/link_4.stl" />
+          <convex_mesh filename="package://abb_irb6700_support/meshes/irb6700_235_265/collision/link_4.stl" convert="true"/>
         </geometry>
         <xacro:material_abb_yellow/>
@@ -127,5 +127,5 @@
         <origin xyz="0 0 0" rpy="0 0 0" />
         <geometry>
-          <mesh filename="package://abb_irb6700_support/meshes/irb6700/collision/link_5.stl" />
+          <convex_mesh filename="package://abb_irb6700_support/meshes/irb6700/collision/link_5.stl" convert="true"/>
         </geometry>
         <xacro:material_abb_yellow/>
@@ -143,5 +143,5 @@
         <origin xyz="0 0 0" rpy="0 0 0" />
         <geometry>
-          <mesh filename="package://abb_irb6700_support/meshes/irb6700/collision/link_6.stl" />
+          <convex_mesh filename="package://abb_irb6700_support/meshes/irb6700/collision/link_6.stl" convert="true"/>
         </geometry>
         <xacro:material_abb_yellow/>

Commit message: Added ability to include calibration offsets

File: abb_irb6700_support/urdf/irb6700_200_260_macro.xacro (robot description, xacro)
@@ -149,6 +149,7 @@
     </link>
     <link name="${prefix}tool0"/>
+    <xacro:property name="cal" value="${load_yaml('$(find abb_irb6700_support)/config/calibration_irb6700_200_260.yaml')}" />
     <joint name="${prefix}joint_1" type="revolute">
-      <origin xyz="0 0 0.78" rpy="0 0 0" />
+      <origin xyz="${0 + cal['j1']['x']} ${0 + cal['j1']['y']} ${0.78 + cal['j1']['z']}" rpy="${0 + cal['j1']['rx']} ${0 + cal['j1']['ry']} ${0 + cal['j1']['rz']}" />
       <parent link="${prefix}base_link" />
       <child link="${prefix}link_1" />
@@ -157,5 +158,6 @@
     </joint>
     <joint name="${prefix}joint_2" type="revolute">
-      <origin xyz="0.32 0 0" rpy="0 0 0" />
+<!--      <origin xyz="0.32 0 0" rpy="0 0 0" />-->
+      <origin xyz="${0.32 + cal['j2']['x']} ${0 + cal['j2']['y']} ${0.0 + cal['j2']['z']}" rpy="${0 + cal['j2']['rx']} ${0 + cal['j2']['ry']} ${0 + cal['j2']['rz']}" />
       <parent link="${prefix}link_1" />
       <child link="${prefix}link_2" />
@@ -164,5 +166,6 @@
     </joint>
     <joint name="${prefix}joint_3" type="revolute">
-      <origin xyz="0 0 1.125" rpy="0 0 0" />
+<!--      <origin xyz="0 0 1.125" rpy="0 0 0" />-->
+      <origin xyz="${0 + cal['j3']['x']} ${0 + cal['j3']['y']} ${1.125 + cal['j3']['z']}" rpy="${0 + cal['j3']['rx']} ${0 + cal['j3']['ry']} ${0 + cal['j3']['rz']}" />
       <parent link="${prefix}link_2" />
       <child link="${prefix}link_3" />
@@ -171,5 +174,6 @@
     </joint>
     <joint name="${prefix}joint_4" type="revolute">
-      <origin xyz="0 0 0.2" rpy="0 0 0" />
+<!--      <origin xyz="0 0 0.2" rpy="0 0 0" />-->
+      <origin xyz="${0 + cal['j4']['x']} ${0 + cal['j4']['y']} ${0.2 + cal['j4']['z']}" rpy="${0 + cal['j4']['rx']} ${0 + cal['j4']['ry']} ${0 + cal['j4']['rz']}" />
       <parent link="${prefix}link_3" />
       <child link="${prefix}link_4" />
@@ -178,5 +182,6 @@
     </joint>
     <joint name="${prefix}joint_5" type="revolute">
-      <origin xyz="1.1425 0 0" rpy="0 0 0" />
+<!--      <origin xyz="1.1425 0 0" rpy="0 0 0" />-->
+      <origin xyz="${1.1425 + cal['j5']['x']} ${0 + cal['j5']['y']} ${0.0 + cal['j5']['z']}" rpy="${0 + cal['j5']['rx']} ${0 + cal['j5']['ry']} ${0 + cal['j5']['rz']}" />
       <parent link="${prefix}link_4" />
       <child link="${prefix}link_5" />
@@ -185,5 +190,6 @@
     </joint>
     <joint name="${prefix}joint_6" type="revolute">
-      <origin xyz="0.2 0 0" rpy="0 0 0" />
+<!--      <origin xyz="0.2 0 0" rpy="0 0 0" />-->
+      <origin xyz="${0.2 + cal['j6']['x']} ${0 + cal['j6']['y']} ${0.0 + cal['j6']['z']}" rpy="${0 + cal['j6']['rx']} ${0 + cal['j6']['ry']} ${0 + cal['j6']['rz']}" />
       <parent link="${prefix}link_5" />
       <child link="${prefix}link_6" />
